Commit message: 优化 URDF 结构 add hangers and lidar pole

File: src/car_description/urdf/car.urdf.xacro (robot description, xacro)
@@ -2,7 +2,9 @@
 <robot xmlns:xacro="http://www.ros.org/wiki/xacro" name="mecanum_car">
   <!--
-    第一版最小可用 URDF：
-    - 重点先把底盘、轮子、IMU、预留雷达坐标系挂起来
-    - 麦轮滚子细节、真实惯量、复杂碰撞先不卷
+    第二版结构增强：
+    - 车体拆成上下板，视觉上不再是一整块实心盒子
+    - 四个轮子补下吊支架
+    - 雷达补安装立柱
+    - 仍然保持最小可用，不在这里硬卷真实机械细节
   -->
   <!-- 车体主体尺寸 -->
@@ -13,4 +15,12 @@
   <xacro:property name="ground_to_body_bottom" value="0.060"/>
   <xacro:property name="base_link_z" value="${ground_to_body_bottom + body_height / 2.0}"/>
+  <!-- 上下板与支撑结构参数 -->
+  <xacro:property name="plate_thickness" value="0.006"/>
+  <xacro:property name="plate_gap" value="${body_height - 2.0 * plate_thickness}"/>
+  <xacro:property name="top_plate_z" value="${body_height / 2.0 - plate_thickness / 2.0}"/>
+  <xacro:property name="bottom_plate_z" value="${-body_height / 2.0 + plate_thickness / 2.0}"/>
+  <xacro:property name="column_size" value="0.012"/>
+  <xacro:property name="column_x" value="0.105"/>
+  <xacro:property name="column_y" value="0.050"/>
   <!-- 轮子参数 -->
   <xacro:property name="wheel_radius" value="0.040"/>
@@ -20,15 +30,28 @@
   <xacro:property name="wheel_x" value="${wheel_base / 2.0}"/>
   <xacro:property name="wheel_y" value="${wheel_track / 2.0}"/>
+  <xacro:property name="wheel_center_z" value="${wheel_radius - base_link_z}"/>
+  <!-- 下吊支架参数 -->
+  <xacro:property name="hanger_x_size" value="0.018"/>
+  <xacro:property name="hanger_y_size" value="0.014"/>
+  <xacro:property name="hanger_drop" value="${bottom_plate_z - wheel_center_z}"/>
+  <xacro:property name="hanger_center_z" value="${(bottom_plate_z + wheel_center_z) / 2.0}"/>
   <!-- 传感器参数 -->
-  <!-- IMU 的 z 按用户给的数据先相对 base_link 保留；这会略高于顶板，后面可再修 -->
   <xacro:property name="imu_x" value="-0.090"/>
   <xacro:property name="imu_y" value="0.0"/>
   <xacro:property name="imu_z" value="0.025"/>
-  <!-- 雷达还没装，这里先放一个不太坑的预留挂点 -->
+  <!-- 雷达还没装，先放一个合理预留位 -->
   <xacro:property name="laser_x" value="0.090"/>
   <xacro:property name="laser_y" value="0.0"/>
   <xacro:property name="laser_z" value="0.090"/>
-  <material name="mat_body">
+  <xacro:property name="laser_radius" value="0.035"/>
+  <xacro:property name="laser_height" value="0.040"/>
+  <xacro:property name="laser_pole_radius" value="0.008"/>
+  <xacro:property name="laser_pole_height" value="${laser_z - top_plate_z - laser_height / 2.0}"/>
+  <xacro:property name="laser_pole_center_z" value="${top_plate_z + laser_pole_height / 2.0}"/>
+  <material name="mat_body_dark">
     <color rgba="0.20 0.20 0.24 1.0"/>
+  </material>
+  <material name="mat_body_light">
+    <color rgba="0.35 0.35 0.40 1.0"/>
   </material>
   <material name="mat_wheel">
@@ -40,4 +63,7 @@
   <material name="mat_laser">
     <color rgba="0.85 0.25 0.15 1.0"/>
+  </material>
+  <material name="mat_support">
+    <color rgba="0.80 0.78 0.68 1.0"/>
   </material>
   <link name="base_footprint"/>
@@ -48,11 +74,51 @@
   </joint>
   <link name="base_link">
-    <visual>
-      <origin xyz="0 0 0" rpy="0 0 0"/>
-      <geometry>
-        <box size="${body_length} ${body_width} ${body_height}"/>
-      </geometry>
-      <material name="mat_body"/>
-    </visual>
+    <!--
+      base_link 仍然作为车体主参考系，但视觉不再用单一大盒子，
+      改为上下板 + 四个立柱，便于看出真实结构层次。
+    -->
+    <visual>
+      <origin xyz="0 0 ${top_plate_z}" rpy="0 0 0"/>
+      <geometry>
+        <box size="${body_length} ${body_width} ${plate_thickness}"/>
+      </geometry>
+      <material name="mat_body_dark"/>
+    </visual>
+    <visual>
+      <origin xyz="0 0 ${bottom_plate_z}" rpy="0 0 0"/>
+      <geometry>
+        <box size="${body_length} ${body_width} ${plate_thickness}"/>
+      </geometry>
+      <material name="mat_body_dark"/>
+    </visual>
+    <visual>
+      <origin xyz="${column_x} ${column_y} 0" rpy="0 0 0"/>
+      <geometry>
+        <box size="${column_size} ${column_size} ${plate_gap}"/>
+      </geometry>
+      <material name="mat_body_light"/>
+    </visual>
+    <visual>
+      <origin xyz="${column_x} ${-column_y} 0" rpy="0 0 0"/>
+      <geometry>
+        <box size="${column_size} ${column_size} ${plate_gap}"/>
+      </geometry>
+      <material name="mat_body_light"/>
+    </visual>
+    <visual>
+      <origin xyz="${-column_x} ${column_y} 0" rpy="0 0 0"/>
+      <geometry>
+        <box size="${column_size} ${column_size} ${plate_gap}"/>
+      </geometry>
+      <material name="mat_body_light"/>
+    </visual>
+    <visual>
+      <origin xyz="${-column_x} ${-column_y} 0" rpy="0 0 0"/>
+      <geometry>
+        <box size="${column_size} ${column_size} ${plate_gap}"/>
+      </geometry>
+      <material name="mat_body_light"/>
+    </visual>
+    <!-- 碰撞先仍然收敛成一个简化盒体，够导航和调 TF 用 -->
     <collision>
       <origin xyz="0 0 0" rpy="0 0 0"/>
@@ -89,31 +155,47 @@
     </link>
   </xacro:macro>
+  <xacro:macro name="wheel_hanger" params="name x y">
+    <link name="${name}">
+      <visual>
+        <origin xyz="0 0 0" rpy="0 0 0"/>
+        <geometry>
+          <box size="${hanger_x_size} ${hanger_y_size} ${hanger_drop}"/>
+        </geometry>
+        <material name="mat_support"/>
+      </visual>
+    </link>
+    <joint name="${name}_joint" type="fixed">
+      <parent link="base_link"/>
+      <child link="${name}"/>
+      <origin xyz="${x} ${y} ${hanger_center_z}" rpy="0 0 0"/>
+    </joint>
+  </xacro:macro>
   <xacro:wheel_link name="front_left_wheel_link"/>
   <xacro:wheel_link name="front_right_wheel_link"/>
   <xacro:wheel_link name="rear_left_wheel_link"/>
   <xacro:wheel_link name="rear_right_wheel_link"/>
-  <!--
-    轮子通过支架下吊，所以 wheel center 会低于车体底板。
-    这里先按给定轴距/轮距挂结构坐标；滚动驱动和真实转向细节后续再接控制层。
-  -->
+  <xacro:wheel_hanger name="front_left_hanger_link" x="${wheel_x}" y="${wheel_y}"/>
+  <xacro:wheel_hanger name="front_right_hanger_link" x="${wheel_x}" y="${-wheel_y}"/>
+  <xacro:wheel_hanger name="rear_left_hanger_link" x="${-wheel_x}" y="${wheel_y}"/>
+  <xacro:wheel_hanger name="rear_right_hanger_link" x="${-wheel_x}" y="${-wheel_y}"/>
   <joint name="front_left_wheel_joint" type="fixed">
     <parent link="base_link"/>
     <child link="front_left_wheel_link"/>
-    <origin xyz="${wheel_x} ${wheel_y} ${wheel_radius - base_link_z}" rpy="0 0 0"/>
+    <origin xyz="${wheel_x} ${wheel_y} ${wheel_center_z}" rpy="0 0 0"/>
   </joint>
   <joint name="front_right_wheel_joint" type="fixed">
     <parent link="base_link"/>
     <child link="front_right_wheel_link"/>
-    <origin xyz="${wheel_x} ${-wheel_y} ${wheel_radius - base_link_z}" rpy="0 0 0"/>
+    <origin xyz="${wheel_x} ${-wheel_y} ${wheel_center_z}" rpy="0 0 0"/>
   </joint>
   <joint name="rear_left_wheel_joint" type="fixed">
     <parent link="base_link"/>
     <child link="rear_left_wheel_link"/>
-    <origin xyz="${-wheel_x} ${wheel_y} ${wheel_radius - base_link_z}" rpy="0 0 0"/>
+    <origin xyz="${-wheel_x} ${wheel_y} ${wheel_center_z}" rpy="0 0 0"/>
   </joint>
   <joint name="rear_right_wheel_joint" type="fixed">
     <parent link="base_link"/>
     <child link="rear_right_wheel_link"/>
-    <origin xyz="${-wheel_x} ${-wheel_y} ${wheel_radius - base_link_z}" rpy="0 0 0"/>
+    <origin xyz="${-wheel_x} ${-wheel_y} ${wheel_center_z}" rpy="0 0 0"/>
   </joint>
   <link name="imu_link">
@@ -130,9 +212,23 @@
     <origin xyz="${imu_x} ${imu_y} ${imu_z}" rpy="0 0 0"/>
   </joint>
+  <link name="laser_pole_link">
+    <visual>
+      <origin xyz="0 0 0" rpy="0 0 0"/>
+      <geometry>
+        <cylinder radius="${laser_pole_radius}" length="${laser_pole_height}"/>
+      </geometry>
+      <material name="mat_support"/>
+    </visual>
+  </link>
+  <joint name="laser_pole_joint" type="fixed">
+    <parent link="base_link"/>
+    <child link="laser_pole_link"/>
+    <origin xyz="${laser_x} ${laser_y} ${laser_pole_center_z}" rpy="0 0 0"/>
+  </joint>
   <link name="laser_link">
     <visual>
       <origin xyz="0 0 0" rpy="0 0 0"/>
       <geometry>
-        <cylinder radius="0.035" length="0.040"/>
+        <cylinder radius="${laser_radius}" length="${laser_height}"/>
       </geometry>
       <material name="mat_laser"/>

Commit message: 修正支架连接 make wheel hangers visibly connected

File: src/car_description/urdf/car.urdf.xacro (robot description, xacro)
@@ -36,4 +36,8 @@
   <xacro:property name="hanger_drop" value="${bottom_plate_z - wheel_center_z}"/>
   <xacro:property name="hanger_center_z" value="${(bottom_plate_z + wheel_center_z) / 2.0}"/>
+  <xacro:property name="outrigger_y_size" value="${wheel_y - body_width / 2.0}"/>
+  <xacro:property name="outrigger_x_size" value="0.030"/>
+  <xacro:property name="outrigger_z_size" value="0.010"/>
+  <xacro:property name="outrigger_center_y" value="${body_width / 2.0 + outrigger_y_size / 2.0}"/>
   <!-- 传感器参数 -->
   <xacro:property name="imu_x" value="-0.090"/>
@@ -155,8 +159,17 @@
     </link>
   </xacro:macro>
-  <xacro:macro name="wheel_hanger" params="name x y">
+  <xacro:macro name="wheel_hanger" params="name x y side_sign">
     <link name="${name}">
+      <!-- 横向外伸连接块：把车体边缘和下吊支架真正接起来 -->
       <visual>
-        <origin xyz="0 0 0" rpy="0 0 0"/>
+        <origin xyz="0 ${side_sign * outrigger_center_y} ${bottom_plate_z}" rpy="0 0 0"/>
+        <geometry>
+          <box size="${outrigger_x_size} ${outrigger_y_size} ${outrigger_z_size}"/>
+        </geometry>
+        <material name="mat_support"/>
+      </visual>
+      <!-- 竖向下吊支架 -->
+      <visual>
+        <origin xyz="0 ${side_sign * outrigger_y_size / 2.0} ${hanger_center_z}" rpy="0 0 0"/>
         <geometry>
           <box size="${hanger_x_size} ${hanger_y_size} ${hanger_drop}"/>
@@ -168,5 +181,5 @@
       <parent link="base_link"/>
       <child link="${name}"/>
-      <origin xyz="${x} ${y} ${hanger_center_z}" rpy="0 0 0"/>
+      <origin xyz="${x} ${side_sign * body_width / 2.0} 0" rpy="0 0 0"/>
     </joint>
   </xacro:macro>
@@ -175,8 +188,8 @@
   <xacro:wheel_link name="rear_left_wheel_link"/>
   <xacro:wheel_link name="rear_right_wheel_link"/>
-  <xacro:wheel_hanger name="front_left_hanger_link" x="${wheel_x}" y="${wheel_y}"/>
-  <xacro:wheel_hanger name="front_right_hanger_link" x="${wheel_x}" y="${-wheel_y}"/>
-  <xacro:wheel_hanger name="rear_left_hanger_link" x="${-wheel_x}" y="${wheel_y}"/>
-  <xacro:wheel_hanger name="rear_right_hanger_link" x="${-wheel_x}" y="${-wheel_y}"/>
+  <xacro:wheel_hanger name="front_left_hanger_link" x="${wheel_x}" y="${wheel_y}" side_sign="1"/>
+  <xacro:wheel_hanger name="front_right_hanger_link" x="${wheel_x}" y="${-wheel_y}" side_sign="-1"/>
+  <xacro:wheel_hanger name="rear_left_hanger_link" x="${-wheel_x}" y="${wheel_y}" side_sign="1"/>
+  <xacro:wheel_hanger name="rear_right_hanger_link" x="${-wheel_x}" y="${-wheel_y}" side_sign="-1"/>
   <joint name="front_left_wheel_joint" type="fixed">
     <parent link="base_link"/>

Commit message: 修正支架位置 fix hanger lateral offset

File: src/car_description/urdf/car.urdf.xacro (robot description, xacro)
@@ -39,5 +39,5 @@
   <xacro:property name="outrigger_x_size" value="0.030"/>
   <xacro:property name="outrigger_z_size" value="0.010"/>
-  <xacro:property name="outrigger_center_y" value="${body_width / 2.0 + outrigger_y_size / 2.0}"/>
+  <xacro:property name="outrigger_center_y" value="${outrigger_y_size / 2.0}"/>
   <!-- 传感器参数 -->
   <xacro:property name="imu_x" value="-0.090"/>
@@ -169,7 +169,7 @@
         <material name="mat_support"/>
       </visual>
-      <!-- 竖向下吊支架 -->
+      <!-- 竖向下吊支架，贴在横向连接块外侧末端 -->
       <visual>
-        <origin xyz="0 ${side_sign * outrigger_y_size / 2.0} ${hanger_center_z}" rpy="0 0 0"/>
+        <origin xyz="0 ${side_sign * (outrigger_y_size + hanger_y_size) / 2.0} ${hanger_center_z}" rpy="0 0 0"/>
         <geometry>
           <box size="${hanger_x_size} ${hanger_y_size} ${hanger_drop}"/>

Commit message: 修正雷达安装位姿 / fix laser_link pose

File: src/car_description/urdf/car.urdf.xacro (robot description, xacro)
@@ -44,8 +44,11 @@
   <xacro:property name="imu_y" value="0.0"/>
   <xacro:property name="imu_z" value="0.025"/>
-  <!-- 雷达还没装，先放一个合理预留位 -->
-  <xacro:property name="laser_x" value="0.090"/>
-  <xacro:property name="laser_y" value="0.0"/>
-  <xacro:property name="laser_z" value="0.090"/>
+  <!-- 当前实装：C1 安装在 base_link 正上方，底部离地约 0.18m；
+       按总高 41.3mm 和扫描窗近中上部估算，扫描平面离地约 0.204m。
+       base_link 几何中心离地约 0.0845m，因此这里先把 laser_link 挂到 z≈0.120m。
+       目前实物前后反装，先用 yaw=pi 修正朝向。 -->
+  <xacro:property name="laser_x" value="0.000"/>
+  <xacro:property name="laser_y" value="0.000"/>
+  <xacro:property name="laser_z" value="0.120"/>
   <xacro:property name="laser_radius" value="0.035"/>
   <xacro:property name="laser_height" value="0.040"/>
@@ -251,5 +254,5 @@
     <parent link="base_link"/>
     <child link="laser_link"/>
-    <origin xyz="${laser_x} ${laser_y} ${laser_z}" rpy="0 0 0"/>
+    <origin xyz="${laser_x} ${laser_y} ${laser_z}" rpy="0 0 3.14159265359"/>
   </joint>
 </robot>

Commit message: 导航与底盘链路整理: nav bringup + odom driver cleanup

File: src/car_description/urdf/car.urdf.xacro (robot description, xacro)
@@ -50,5 +50,5 @@
   <xacro:property name="laser_x" value="0.000"/>
   <xacro:property name="laser_y" value="0.000"/>
-  <xacro:property name="laser_z" value="0.120"/>
+  <xacro:property name="laser_z" value="0.080"/>
   <xacro:property name="laser_radius" value="0.035"/>
   <xacro:property name="laser_height" value="0.040"/>

Commit message: 添加深度相机

File: src/car_description/urdf/car.urdf.xacro (robot description, xacro)
@@ -74,4 +74,16 @@
     <color rgba="0.80 0.78 0.68 1.0"/>
   </material>
+  <!-- 相机参数：Astra Pro 当前装在车头，后侧紧贴车体前缘，顶部与上车板上表面齐平。
+       这里先按外壳近似尺寸建模，重点是把 camera_link / optical frame 挂进 TF。 -->
+  <xacro:property name="camera_x_size" value="0.030"/>
+  <xacro:property name="camera_y_size" value="0.165"/>
+  <xacro:property name="camera_z_size" value="0.040"/>
+  <xacro:property name="camera_x" value="${body_length / 2.0 + camera_x_size / 2.0}"/>
+  <xacro:property name="camera_y" value="0.0"/>
+  <xacro:property name="camera_z" value="${body_height / 2.0 - camera_z_size / 2.0}"/>
+  <xacro:property name="camera_optical_x" value="${camera_x_size / 2.0}"/>
+  <material name="mat_camera">
+    <color rgba="0.05 0.05 0.06 1.0"/>
+  </material>
   <link name="base_footprint"/>
   <joint name="base_footprint_to_base_link" type="fixed">
@@ -256,3 +268,48 @@
     <origin xyz="${laser_x} ${laser_y} ${laser_z}" rpy="0 0 3.14159265359"/>
   </joint>
+  <link name="camera_link">
+    <visual>
+      <origin xyz="0 0 0" rpy="0 0 0"/>
+      <geometry>
+        <box size="${camera_x_size} ${camera_y_size} ${camera_z_size}"/>
+      </geometry>
+      <material name="mat_camera"/>
+    </visual>
+    <collision>
+      <origin xyz="0 0 0" rpy="0 0 0"/>
+      <geometry>
+        <box size="${camera_x_size} ${camera_y_size} ${camera_z_size}"/>
+      </geometry>
+    </collision>
+  </link>
+  <joint name="camera_joint" type="fixed">
+    <parent link="base_link"/>
+    <child link="camera_link"/>
+    <origin xyz="${camera_x} ${camera_y} ${camera_z}" rpy="0 0 0"/>
+  </joint>
+  <!-- Orbbec 常用帧：深度和彩色帧从 camera_link 展开，optical frame 遵循 REP-103：z 向前，x 向右，y 向下。 -->
+  <link name="camera_depth_frame"/>
+  <joint name="camera_depth_joint" type="fixed">
+    <parent link="camera_link"/>
+    <child link="camera_depth_frame"/>
+    <origin xyz="${camera_optical_x} 0 0" rpy="0 0 0"/>
+  </joint>
+  <link name="camera_depth_optical_frame"/>
+  <joint name="camera_depth_optical_joint" type="fixed">
+    <parent link="camera_depth_frame"/>
+    <child link="camera_depth_optical_frame"/>
+    <origin xyz="0 0 0" rpy="-1.57079632679 0 -1.57079632679"/>
+  </joint>
+  <link name="camera_color_frame"/>
+  <joint name="camera_color_joint" type="fixed">
+    <parent link="camera_link"/>
+    <child link="camera_color_frame"/>
+    <origin xyz="${camera_optical_x} 0 0" rpy="0 0 0"/>
+  </joint>
+  <link name="camera_color_optical_frame"/>
+  <joint name="camera_color_optical_joint" type="fixed">
+    <parent link="camera_color_frame"/>
+    <child link="camera_color_optical_frame"/>
+    <origin xyz="0 0 0" rpy="-1.57079632679 0 -1.57079632679"/>
+  </joint>
 </robot>
